File: tiny328-wifirelay.kicad_pcb (KiCad board)
At the start: 2 copper layers, 35.4 x 25.2 mm, 8 parts, among them P1 RX868SH-DV, U1 TINY328, U2 ESP-01v090, U3 LD1117S33TR

Commit message: updated for PCB run #1
Parts:
- added D1: LED, LEDs:LED-0805, F.Cu at (133.6, 102.4)
- added D2: LED, LEDs:LED-0805, F.Cu at (133.6, 104.3)
- added D3: LED, LEDs:LED-0805, F.Cu at (133.6, 106.2)
- added D4: LED, LEDs:LED-0805, F.Cu at (133.6, 108.1)
- added R2: 68, Resistors_SMD:R_0603_HandSoldering, F.Cu at (137.8, 102.4)
- added R3: 68, Resistors_SMD:R_0603_HandSoldering, F.Cu at (137.8, 104.3)
- added R4: 68, Resistors_SMD:R_0603_HandSoldering, F.Cu at (137.8, 106.2)
- added R5: 68, Resistors_SMD:R_0603_HandSoldering, F.Cu at (137.8, 108.1)
Routing:
- net GND: track 51.8 -> 79.2 mm
- net Net-(R2-Pad2): track 0.00 -> 21.2 mm
- net Net-(R3-Pad2): track 0.00 -> 18.5 mm
- net /ESP_RX: track 23.2 -> 36.9 mm
- net Net-(R4-Pad2): track 0.00 -> 12.7 mm
- net Net-(R5-Pad2): track 0.00 -> 9.55 mm
- net Net-(D4-Pad1): track 0.00 -> 2.05 mm
- net Net-(D3-Pad1): track 0.00 -> 2.05 mm
- net Net-(D2-Pad1): track 0.00 -> 2.05 mm
- net Net-(D1-Pad1): track 0.00 -> 2.05 mm
- net +3V3: track 81.3 -> 82.4 mm
- net +5V: track 18.6 -> 19.4 mm
- added copper zone on B.Cu, net +3V3
- added copper zone on F.Cu, net GND
